Commit message: gazebo_fix

File: install/catatron_description/share/catatron_description/urdf/catatron.urdf (robot description, URDF)
Before this commit: robot catatron, 22 links, 21 joints
Links:
- link base_link: geometry collision box size=0.260 0.160 0.090; visual mesh filename=file:///home/abhinand/Envisage/catatron_ws/src/catatron_des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
- link femur_bl_link: geometry collision box size=0.040 0.070 0.130; visual mesh filename=file:///home/abhinand/Envisage/catatron_ws/src/catatron_des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
- link femur_br_link: geometry collision box size=0.040 0.070 0.130; visual mesh filename=file:///home/abhinand/Envisage/catatron_ws/src/catatron_des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
- link femur_fl_link: geometry collision box size=0.040 0.070 0.130; visual mesh filename=file:///home/abhinand/Envisage/catatron_ws/src/catatron_des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
- link femur_fr_link: geometry collision box size=0.040 0.070 0.130; visual mesh filename=file:///home/abhinand/Envisage/catatron_ws/src/catatron_des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
- link hip_bl_link: geometry collision box size=0.050 0.050 0.070; visual mesh filename=file:///home/abhinand/Envisage/catatron_ws/src/catatron_des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
- link hip_bl_ref: mass 0.000 -> 0.001
- link hip_br_link: geometry collision box size=0.050 0.050 0.070; visual mesh filename=file:///home/abhinand/Envisage/catatron_ws/src/catatron_des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
- link hip_br_ref: mass 0.000 -> 0.001
- link hip_fl_link: geometry collision box size=0.050 0.050 0.070; visual mesh filename=file:///home/abhinand/Envisage/catatron_ws/src/catatron_des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
- link hip_fl_ref: mass 0.000 -> 0.001
- link hip_fr_link: geometry collision box size=0.050 0.050 0.070; visual mesh filename=file:///home/abhinand/Envisage/catatron_ws/src/catatron_des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
- link hip_fr_ref: mass 0.000 -> 0.001
- link lidar_link: geometry collision box size=0.080 0.060 0.050; visual mesh filename=file:///home/abhinand/Envisage/catatron_ws/src/catatron_des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
- link tibia_bl_link: geometry visual mesh filename=file:///home/abhinand/Envisage/catatron_ws/src/catatron_des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
- link tibia_br_link: geometry visual mesh filename=file:///home/abhinand/Envisage/catatron_ws/src/catatron_des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
- link tibia_fl_link: geometry visual mesh filename=file:///home/abhinand/Envisage/catatron_ws/src/catatron_des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
- link tibia_fr_link: geometry visual mesh filename=file:///home/abhinand/Envisage/catatron_ws/src/catatron_des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

Commit message: inv-kin

File: install/catatron_description/share/catatron_description/urdf/catatron.urdf (robot description, URDF)
Before this commit: robot catatron, 22 links, 21 joints
Links:
- link base_link: geometry collision box size=0.260 0.160 0.090; visual mesh filename=/home/abhinand/Envisage/catatron_ws/src/catatron_descriptio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
- link femur_bl_link: geometry collision box size=0.040 0.070 0.110; visual mesh filename=/home/abhinand/Envisage/catatron_ws/src/catatron_descriptio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
- link femur_br_link: geometry collision box size=0.040 0.070 0.110; visual mesh filename=/home/abhinand/Envisage/catatron_ws/src/catatron_descriptio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
- link femur_fl_link: geometry collision box size=0.040 0.070 0.110; visual mesh filename=/home/abhinand/Envisage/catatron_ws/src/catatron_descriptio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
- link femur_fr_link: geometry collision box size=0.040 0.070 0.110; visual mesh filename=/home/abhinand/Envisage/catatron_ws/src/catatron_descriptio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
- link hip_bl_link: geometry collision box size=0.050 0.050 0.070; visual mesh filename=/home/abhinand/Envisage/catatron_ws/src/catatron_descriptio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
- link hip_br_link: geometry collision box size=0.050 0.050 0.070; visual mesh filename=/home/abhinand/Envisage/catatron_ws/src/catatron_descriptio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
- link hip_fl_link: geometry collision box size=0.050 0.050 0.070; visual mesh filename=/home/abhinand/Envisage/catatron_ws/src/catatron_descriptio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
- link hip_fr_link: geometry collision box size=0.050 0.050 0.070; visual mesh filename=/home/abhinand/Envisage/catatron_ws/src/catatron_descriptio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
- link lidar_link: geometry collision box size=0.080 0.060 0.050; visual mesh filename=/home/abhinand/Envisage/catatron_ws/src/catatron_descriptio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
- link tibia_bl_link: geometry collision box size=0.040 0.070 0.110; visual mesh filename=/home/abhinand/Envisage/catatron_ws/src/catatron_descriptio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
- link tibia_br_link: geometry collision box size=0.040 0.070 0.110; visual mesh filename=/home/abhinand/Envisage/catatron_ws/src/catatron_descriptio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
- link tibia_fl_link: geometry collision box size=0.040 0.070 0.110; visual mesh filename=/home/abhinand/Envisage/catatron_ws/src/catatron_descriptio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
- link tibia_fr_link: geometry collision box size=0.040 0.070 0.110; visual mesh filename=/home/abhinand/Envisage/catatron_ws/src/catatron_descriptio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

Commit message: stand_pose

File: install/catatron_description/share/catatron_description/urdf/catatron.urdf (robot description, URDF)
Before this commit: robot catatron, 22 links, 21 joints
Links:
- removed link lidar_link
Joints:
- removed joint lidar

Commit message: imu control

File: install/catatron_description/share/catatron_description/urdf/catatron.urdf (robot description, URDF)
Before this commit: robot catatron, 21 links, 20 joints
Links:
- added link imu_link, mass 0.05; collision box size=0.05 0.05 0.01; visual box size=0.05 0.05 0.01
- link base_link: geometry collision mesh filename=/home/abhinand/Envisage/catatron_ws/src/catatron_descriptio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; visual mesh filename=/home/abhinand/Envisage/catatron_ws/src/catatron_descriptio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
- link femur_bl_link: geometry collision mesh filename=/home/abhinand/Envisage/catatron_ws/src/catatron_descriptio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; visual mesh filename=/home/abhinand/Envisage/catatron_ws/src/catatron_descriptio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
- link femur_br_link: geometry collision mesh filename=/home/abhinand/Envisage/catatron_ws/src/catatron_descriptio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; visual mesh filename=/home/abhinand/Envisage/catatron_ws/src/catatron_descriptio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
- link femur_fl_link: geometry collision mesh filename=/home/abhinand/Envisage/catatron_ws/src/catatron_descriptio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; visual mesh filename=/home/abhinand/Envisage/catatron_ws/src/catatron_descriptio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
- link femur_fr_link: geometry collision mesh filename=/home/abhinand/Envisage/catatron_ws/src/catatron_descriptio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; visual mesh filename=/home/abhinand/Envisage/catatron_ws/src/catatron_descriptio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
- link hip_bl_link: geometry collision mesh filename=/home/abhinand/Envisage/catatron_ws/src/catatron_descriptio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; visual mesh filename=/home/abhinand/Envisage/catatron_ws/src/catatron_descriptio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
- link hip_br_link: geometry collision mesh filename=/home/abhinand/Envisage/catatron_ws/src/catatron_descriptio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; visual mesh filename=/home/abhinand/Envisage/catatron_ws/src/catatron_descriptio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
- link hip_fl_link: geometry collision mesh filename=/home/abhinand/Envisage/catatron_ws/src/catatron_descriptio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; visual mesh filename=/home/abhinand/Envisage/catatron_ws/src/catatron_descriptio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
- link hip_fr_link: geometry collision mesh filename=/home/abhinand/Envisage/catatron_ws/src/catatron_descriptio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; visual mesh filename=/home/abhinand/Envisage/catatron_ws/src/catatron_descriptio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
- link tibia_bl_link: geometry collision mesh filename=/home/abhinand/Envisage/catatron_ws/src/catatron_descriptio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; visual mesh filename=/home/abhinand/Envisage/catatron_ws/src/catatron_descriptio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
- link tibia_br_link: geometry collision mesh filename=/home/abhinand/Envisage/catatron_ws/src/catatron_descriptio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; visual mesh filename=/home/abhinand/Envisage/catatron_ws/src/catatron_descriptio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
- link tibia_fl_link: geometry collision mesh filename=/home/abhinand/Envisage/catatron_ws/src/catatron_descriptio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; visual mesh filename=/home/abhinand/Envisage/catatron_ws/src/catatron_descriptio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
- link tibia_fr_link: geometry collision mesh filename=/home/abhinand/Envisage/catatron_ws/src/catatron_descriptio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; visual mesh filename=/home/abhinand/Envisage/catatron_ws/src/catatron_descriptio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
Joints:
- added joint imu_joint: type fixed, parent base_link, child imu_link, origin xyz=0.0 0.0 0.06 rpy=0 0 0
- joint hip1_bl: limit lower=-0.78540 upper=1.57080 effort=80.00000 velocity=1.04720 -> lower=-3.142 upper=3.142 effort=80.00000 velocity=1.04720
- joint hip1_br: limit lower=-0.78540 upper=1.57080 effort=80.00000 velocity=1.04720 -> lower=-3.142 upper=3.142 effort=80.00000 velocity=1.04720
- joint hip1_fl: limit lower=-0.78540 upper=1.57080 effort=80.00000 velocity=1.04720 -> lower=-3.142 upper=3.142 effort=80.00000 velocity=1.04720
- joint hip1_fr: limit lower=-0.78540 upper=1.57080 effort=80.00000 velocity=1.04720 -> lower=-3.142 upper=3.142 effort=80.00000 velocity=1.04720
- joint hip2_bl: limit lower=0.00000 upper=2.35619 effort=80.00000 velocity=1.04720 -> lower=-3.142 upper=3.142 effort=80.00000 velocity=1.04720
- joint hip2_br: limit lower=0.00000 upper=2.35619 effort=80.00000 velocity=1.04720 -> lower=-3.142 upper=3.142 effort=80.00000 velocity=1.04720
- joint hip2_fl: limit lower=0.00000 upper=2.35619 effort=80.00000 velocity=1.04720 -> lower=-3.142 upper=3.142 effort=80.00000 velocity=1.04720
- joint hip2_fr: limit lower=0.00000 upper=2.35619 effort=80.00000 velocity=1.04720 -> lower=-3.142 upper=3.142 effort=80.00000 velocity=1.04720
- joint knee_bl: limit lower=-2.35619 upper=-0.52360 effort=80.00000 velocity=1.04720 -> lower=-3.142 upper=-0.52360 effort=80.00000 velocity=1.04720
- joint knee_br: limit lower=-2.35619 upper=-0.52360 effort=80.00000 velocity=1.04720 -> lower=-3.142 upper=-0.52360 effort=80.00000 velocity=1.04720
- joint knee_fl: limit lower=-2.35619 upper=-0.52360 effort=80.00000 velocity=1.04720 -> lower=-3.142 upper=-0.52360 effort=80.00000 velocity=1.04720
- joint knee_fr: limit lower=-2.35619 upper=-0.52360 effort=80.00000 velocity=1.04720 -> lower=-3.142 upper=-0.52360 effort=80.00000 velocity=1.04720

Commit message: converted to dae

File: install/catatron_description/share/catatron_description/urdf/catatron.urdf (robot description, URDF)
Before this commit: robot catatron, 22 links, 21 joints
Links:
- removed link feet_bl
- removed link feet_br
- removed link feet_fl
- removed link feet_fr
- removed link femur_bl_link
- removed link femur_br_link
- removed link femur_fl_link
- removed link femur_fr_link
- removed link hip_bl_link
- removed link hip_bl_ref
- removed link hip_br_link
- removed link hip_br_ref
- removed link hip_fl_link
- removed link hip_fl_ref
- removed link hip_fr_link
- removed link hip_fr_ref
- removed link tibia_bl_link
- removed link tibia_br_link
- removed link tibia_fl_link
- removed link tibia_fr_link
- added link FL1, mass 0.15334; visual mesh filename=package://catatron_description/mesh_files/FL1_obj.dae
- added link FL2, mass 0.15106; collision cylinder length=0.125 radius=0.014; visual mesh filename=package://catatron_description/mesh_files/L2_obj.dae
- added link FL3, mass 0.023372; collision cylinder length=0.06 radius=0.007; visual mesh filename=package://catatron_description/mesh_files/L3_obj.dae
- added link FL4, mass 0.0391; collision sphere radius=0.0072
- added link FR1, mass 0.15379; visual mesh filename=package://catatron_description/mesh_files/FR1_obj.dae
- added link FR2, mass 0.15106; collision cylinder length=0.125 radius=0.014; visual mesh filename=package://catatron_description/mesh_files/R2_obj.dae
- added link FR3, mass 0.023372; collision cylinder length=0.06 radius=0.007; visual mesh filename=package://catatron_description/mesh_files/R3_obj.dae
- added link FR4, mass 0.0391; collision sphere radius=0.0072
- added link RL1, mass 0.15379; visual mesh filename=package://catatron_catatron_description/mesh_files/RL1_obj.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
- added link RL2, mass 0.15106; collision cylinder length=0.125 radius=0.014; visual mesh filename=package://catatron_description/mesh_files/L2_obj.dae
- added link RL3, mass 0.023372; collision cylinder length=0.06 radius=0.007; visual mesh filename=package://catatron_description/mesh_files/L3_obj.dae
- added link RL4, mass 0.0391; collision sphere radius=0.0072
- added link RR1, mass 0.15379; visual mesh filename=package://catatron_description/mesh_files/RR1_obj.dae
- added link RR2, mass 0.15106; collision cylinder length=0.125 radius=0.014; visual mesh filename=package://catatron_description/mesh_files/R2_obj.dae
- added link RR3, mass 0.023372; collision cylinder length=0.06 radius=0.007; visual mesh filename=package://catatron_description/mesh_files/R3_obj.dae
- added link RR4, mass 0.0391; collision sphere radius=0.0072
- link base_link: mass 2.000 -> 0.81776; geometry collision box size=0.25 0.1285 0.055; visual mesh filename=package://catatron_description/mesh_files/body_obj.dae
Joints:
- removed joint bl_ref
- removed joint br_ref
- removed joint feet_bl_ref
- removed joint feet_br_ref
- removed joint feet_fl_ref
- removed joint feet_fr_ref
- removed joint fl_ref
- removed joint fr_ref
- removed joint hip1_bl
- removed joint hip1_br
- removed joint hip1_fl
- removed joint hip1_fr
- removed joint hip2_bl
- removed joint hip2_br
- removed joint hip2_fl
- removed joint hip2_fr
- removed joint knee_bl
- removed joint knee_br
- removed joint knee_fl
- removed joint knee_fr
- added joint FL1_joint: type revolute, parent base_link, child FL1, origin xyz=0.0954 0.04 0 rpy=1.5708 0 -1.5708, axis 0 0 1, limit lower=-3 upper=3 effort=1.4 velocity=3
- added joint FL2_joint: type revolute, parent FL1, child FL2, origin xyz=-0.0469 0 0 rpy=1.5708 0 -1.5708, axis 0 0 1, limit lower=-3 upper=3 effort=1.4 velocity=3
- added joint FL3_joint: type revolute, parent FL2, child FL3, origin xyz=0.1 0 0 rpy=0 0 0, axis 0 0 1, limit lower=-3 upper=3 effort=1.4 velocity=3
- added joint FL4_joint: type fixed, parent FL3, child FL4, origin xyz=0.094333 0 0 rpy=0 0 0, axis 0 0 0
- added joint FR1_joint: type revolute, parent base_link, child FR1, origin xyz=0.0954 -0.04 0 rpy=1.5708 0 -1.5708, axis 0 0 1, limit lower=-3 upper=3 effort=1.4 velocity=3
- added joint FR2_joint: type revolute, parent FR1, child FR2, origin xyz=0.0469 0 0 rpy=1.5708 0 -1.5708, axis 0 0 1, limit lower=-3 upper=3 effort=1.4 velocity=3
- added joint FR3_joint: type revolute, parent FR2, child FR3, origin xyz=0.1 0 0 rpy=0 0 0, axis 0 0 1, limit lower=-3 upper=3 effort=1.4 velocity=3
- added joint FR4_joint: type fixed, parent FR3, child FR4, origin xyz=0.094333 0 0 rpy=0 0 0, axis 0 0 0
- added joint RL1_joint: type revolute, parent base_link, child RL1, origin xyz=-0.0954 0.04 0 rpy=1.5708 0 -1.5708, axis 0 0 1, limit lower=-3 upper=3 effort=1.4 velocity=3
- added joint RL2_joint: type revolute, parent RL1, child RL2, origin xyz=-0.0469 0 0 rpy=1.5708 0 -1.5708, axis 0 0 1, limit lower=-3 upper=3 effort=1.4 velocity=3
- added joint RL3_joint: type revolute, parent RL2, child RL3, origin xyz=0.1 0 0 rpy=0 0 0, axis 0 0 1, limit lower=-3 upper=3 effort=1.4 velocity=3
- added joint RL4_joint: type fixed, parent RL3, child RL4, origin xyz=0.094333 0 0 rpy=0 0 0, axis 0 0 0
- added joint RR1_joint: type revolute, parent base_link, child RR1, origin xyz=-0.0954 -0.04 0 rpy=1.5708 0 -1.5708, axis 0 0 1, limit lower=-3 upper=3 effort=1.4 velocity=3
- added joint RR2_joint: type revolute, parent RR1, child RR2, origin xyz=0.0469 0 0 rpy=1.5708 0 -1.5708, axis 0 0 1, limit lower=-3 upper=3 effort=1.4 velocity=3
- added joint RR3_joint: type revolute, parent RR2, child RR3, origin xyz=0.1 0 0 rpy=0 0 0, axis 0 0 1, limit lower=-3 upper=3 effort=1.4 velocity=3
- added joint RR4_joint: type fixed, parent RR3, child RR4, origin xyz=0.094333 0 0 rpy=0 0 0, axis 0 0 0

File: src/catatron_description/urdf/catatron.urdf (robot description, URDF)
Before this commit: robot catatron, 18 links, 17 joints
Links:
- removed link world
- added link imu_link, mass 0.05; collision box size=0.05 0.05 0.01; visual box size=0.05 0.05 0.01
- link FL1: geometry visual mesh filename=package://catatron_description/mesh_files/FL1_obj.dae
- link FL2: geometry collision cylinder length=0.125 radius=0.014; visual mesh filename=package://catatron_description/mesh_files/L2_obj.dae
- link FL3: geometry collision cylinder length=0.06 radius=0.007; visual mesh filename=package://catatron_description/mesh_files/L3_obj.dae
- link FR1: geometry visual mesh filename=package://catatron_description/mesh_files/FR1_obj.dae
- link FR2: geometry collision cylinder length=0.125 radius=0.014; visual mesh filename=package://catatron_description/mesh_files/R2_obj.dae
- link FR3: geometry collision cylinder length=0.06 radius=0.007; visual mesh filename=package://catatron_description/mesh_files/R3_obj.dae
- link RL2: geometry collision cylinder length=0.125 radius=0.014; visual mesh filename=package://catatron_description/mesh_files/L2_obj.dae
- link RL3: geometry collision cylinder length=0.06 radius=0.007; visual mesh filename=package://catatron_description/mesh_files/L3_obj.dae
- link RR1: geometry visual mesh filename=package://catatron_description/mesh_files/RR1_obj.dae
- link RR2: geometry collision cylinder length=0.125 radius=0.014; visual mesh filename=package://catatron_description/mesh_files/R2_obj.dae
- link RR3: geometry collision cylinder length=0.06 radius=0.007; visual mesh filename=package://catatron_description/mesh_files/R3_obj.dae
- link base_link: geometry collision box size=0.25 0.1285 0.055; visual mesh filename=package://catatron_description/mesh_files/body_obj.dae
Joints:
- removed joint world_to_base
- added joint imu_joint: type fixed, parent base_link, child imu_link, origin xyz=0.0 0.0 0.06 rpy=0 0 0
