Commit message: fixed resource manager

File: install/catatron_description/share/catatron_description/urdf/catatron.urdf (robot description, URDF)
Before this commit: robot catatron, 18 links, 17 joints
Links:
- removed link FL1
- removed link FL2
- removed link FL3
- removed link FL4
- removed link FR1
- removed link FR2
- removed link FR3
- removed link FR4
- removed link RL1
- removed link RL2
- removed link RL3
- removed link RL4
- removed link RR1
- removed link RR2
- removed link RR3
- removed link RR4
- removed link world
- added link feet_bl, mass 0.010; collision box size=0.011 0.011 0.011; visual sphere radius=0.001
- added link feet_br, mass 0.010; collision box size=0.011 0.011 0.011; visual sphere radius=0.001
- added link feet_fl, mass 0.010; collision box size=0.011 0.011 0.011; visual sphere radius=0.001
- added link feet_fr, mass 0.010; collision box size=0.011 0.011 0.011; visual sphere radius=0.001
- added link femur_bl_link, mass 0.084; collision mesh filename=/home/ajoymathew07/Catatron/Catatron/src/catatron_descripti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; visual mesh filename=/home/ajoymathew07/Catatron/Catatron/src/catatron_descripti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
- added link femur_br_link, mass 0.084; collision mesh filename=/home/ajoymathew07/Catatron/Catatron/src/catatron_descripti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; visual mesh filename=/home/ajoymathew07/Catatron/Catatron/src/catatron_descripti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
- added link femur_fl_link, mass 0.084; collision mesh filename=/home/ajoymathew07/Catatron/Catatron/src/catatron_descripti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; visual mesh filename=/home/ajoymathew07/Catatron/Catatron/src/catatron_descripti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
- added link femur_fr_link, mass 0.084; collision mesh filename=/home/ajoymathew07/Catatron/Catatron/src/catatron_descripti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; visual mesh filename=/home/ajoymathew07/Catatron/Catatron/src/catatron_descripti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
- added link hip_bl_link, mass 0.233; collision mesh filename=/home/ajoymathew07/Catatron/Catatron/src/catatron_descripti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; visual mesh filename=/home/ajoymathew07/Catatron/Catatron/src/catatron_descripti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
- added link hip_bl_ref, mass 0.001; collision box size=0.002 0.002 0.002; visual box size=0.002 0.002 0.002
- added link hip_br_link, mass 0.233; collision mesh filename=/home/ajoymathew07/Catatron/Catatron/src/catatron_descripti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; visual mesh filename=/home/ajoymathew07/Catatron/Catatron/src/catatron_descripti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
- added link hip_br_ref, mass 0.001; collision box size=0.002 0.002 0.002; visual box size=0.002 0.002 0.002
- added link hip_fl_link, mass 0.233; collision mesh filename=/home/ajoymathew07/Catatron/Catatron/src/catatron_descripti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; visual mesh filename=/home/ajoymathew07/Catatron/Catatron/src/catatron_descripti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
- added link hip_fl_ref, mass 0.001; collision box size=0.002 0.002 0.002; visual box size=0.002 0.002 0.002
- added link hip_fr_link, mass 0.233; collision mesh filename=/home/ajoymathew07/Catatron/Catatron/src/catatron_descripti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; visual mesh filename=/home/ajoymathew07/Catatron/Catatron/src/catatron_descripti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
- added link hip_fr_ref, mass 0.001; collision box size=0.002 0.002 0.002; visual box size=0.002 0.002 0.002
- added link imu_link, mass 0.05; collision box size=0.05 0.05 0.01; visual box size=0.05 0.05 0.01
- added link tibia_bl_link, mass 0.034; collision mesh filename=/home/ajoymathew07/Catatron/Catatron/src/catatron_descripti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; visual mesh filename=/home/ajoymathew07/Catatron/Catatron/src/catatron_descripti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
- added link tibia_br_link, mass 0.034; collision mesh filename=/home/ajoymathew07/Catatron/Catatron/src/catatron_descripti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; visual mesh filename=/home/ajoymathew07/Catatron/Catatron/src/catatron_descripti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
- added link tibia_fl_link, mass 0.034; collision mesh filename=/home/ajoymathew07/Catatron/Catatron/src/catatron_descripti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; visual mesh filename=/home/ajoymathew07/Catatron/Catatron/src/catatron_descripti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
- added link tibia_fr_link, mass 0.034; collision mesh filename=/home/ajoymathew07/Catatron/Catatron/src/catatron_descripti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; visual mesh filename=/home/ajoymathew07/Catatron/Catatron/src/catatron_descripti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
- link base_link: mass 0.81776 -> 2.000; geometry collision mesh filename=/home/ajoymathew07/Catatron/Catatron/src/catatron_descripti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; visual mesh filename=/home/ajoymathew07/Catatron/Catatron/src/catatron_descripti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
Joints:
- removed joint FL1_joint
- removed joint FL2_joint
- removed joint FL3_joint
- removed joint FL4_joint
- removed joint FR1_joint
- removed joint FR2_joint
- removed joint FR3_joint
- removed joint FR4_joint
- removed joint RL1_joint
- removed joint RL2_joint
- removed joint RL3_joint
- removed joint RL4_joint
- removed joint RR1_joint
- removed joint RR2_joint
- removed joint RR3_joint
- removed joint RR4_joint
- removed joint world_to_base
- added joint bl_ref: type fixed, parent base_link, child hip_bl_ref, origin xyz=-0.09170 0.05355 -0.00279
- added joint br_ref: type fixed, parent base_link, child hip_br_ref, origin xyz=-0.09170 -0.05355 -0.00279
- added joint feet_bl_ref: type fixed, parent tibia_bl_link, child feet_bl, origin xyz=0.00000 -0.00834 -0.10000
- added joint feet_br_ref: type fixed, parent tibia_br_link, child feet_br, origin xyz=0.00000 0.00834 -0.10000
- added joint feet_fl_ref: type fixed, parent tibia_fl_link, child feet_fl, origin xyz=0.00000 -0.00834 -0.10000
- added joint feet_fr_ref: type fixed, parent tibia_fr_link, child feet_fr, origin xyz=0.00000 0.00834 -0.10000
- added joint fl_ref: type fixed, parent base_link, child hip_fl_ref, origin xyz=0.09170 0.05355 -0.00279
- added joint fr_ref: type fixed, parent base_link, child hip_fr_ref, origin xyz=0.09170 -0.05355 -0.00279
- added joint hip1_bl: type revolute, parent hip_bl_ref, child hip_bl_link, origin xyz=0.00000 0.00000 0.00000, axis 1.000 0.000 0.000, limit lower=-3.142 upper=3.142 effort=80.00000 velocity=1.04720
- added joint hip1_br: type revolute, parent hip_br_ref, child hip_br_link, origin xyz=0.00000 0.00000 0.00000, axis 1.000 0.000 0.000, limit lower=-3.142 upper=3.142 effort=80.00000 velocity=1.04720
- added joint hip1_fl: type revolute, parent hip_fl_ref, child hip_fl_link, origin xyz=0.00000 0.00000 0.00000, axis 1.000 0.000 0.000, limit lower=-3.142 upper=3.142 effort=80.00000 velocity=1.04720
- added joint hip1_fr: type revolute, parent hip_fr_ref, child hip_fr_link, origin xyz=0.00000 0.00000 0.00000, axis 1.000 0.000 0.000, limit lower=-3.142 upper=3.142 effort=80.00000 velocity=1.04720
- added joint hip2_bl: type revolute, parent hip_bl_link, child femur_bl_link, origin xyz=0.00000 0.03559 0.00000, axis 0.000 1.000 0.000, limit lower=-3.142 upper=3.142 effort=80.00000 velocity=1.04720
- added joint hip2_br: type revolute, parent hip_br_link, child femur_br_link, origin xyz=0.00000 -0.03559 0.00000, axis 0.000 1.000 0.000, limit lower=-3.142 upper=3.142 effort=80.00000 velocity=1.04720
- added joint hip2_fl: type revolute, parent hip_fl_link, child femur_fl_link, origin xyz=0.00000 0.03559 0.00000, axis 0.000 1.000 0.000, limit lower=-3.142 upper=3.142 effort=80.00000 velocity=1.04720
- added joint hip2_fr: type revolute, parent hip_fr_link, child femur_fr_link, origin xyz=0.00000 -0.03559 0.00000, axis 0.000 1.000 0.000, limit lower=-3.142 upper=3.142 effort=80.00000 velocity=1.04720
- added joint imu_joint: type fixed, parent base_link, child imu_link, origin xyz=0.0 0.0 0.06 rpy=0 0 0
- added joint knee_bl: type revolute, parent femur_bl_link, child tibia_bl_link, origin xyz=0.00000 0.01071 -0.09996, axis 0.000 1.000 0.000, limit lower=-3.142 upper=-0.52360 effort=80.00000 velocity=1.04720
- added joint knee_br: type revolute, parent femur_br_link, child tibia_br_link, origin xyz=0.00000 -0.01071 -0.09996, axis 0.000 1.000 0.000, limit lower=-3.142 upper=-0.52360 effort=80.00000 velocity=1.04720
- added joint knee_fl: type revolute, parent femur_fl_link, child tibia_fl_link, origin xyz=0.00000 0.01071 -0.09996, axis 0.000 1.000 0.000, limit lower=-3.142 upper=-0.52360 effort=80.00000 velocity=1.04720
- added joint knee_fr: type revolute, parent femur_fr_link, child tibia_fr_link, origin xyz=0.00000 -0.01071 -0.09996, axis 0.000 1.000 0.000, limit lower=-3.142 upper=-0.52360 effort=80.00000 velocity=1.04720

File: src/catatron_description/urdf/catatron.urdf (robot description, URDF)
Before this commit: robot catatron, 18 links, 17 joints
Links:
- removed link FL1
- removed link FL2
- removed link FL3
- removed link FL4
- removed link FR1
- removed link FR2
- removed link FR3
- removed link FR4
- removed link RL1
- removed link RL2
- removed link RL3
- removed link RL4
- removed link RR1
- removed link RR2
- removed link RR3
- removed link RR4
- removed link world
- added link feet_bl, mass 0.010; collision box size=0.011 0.011 0.011; visual sphere radius=0.001
- added link feet_br, mass 0.010; collision box size=0.011 0.011 0.011; visual sphere radius=0.001
- added link feet_fl, mass 0.010; collision box size=0.011 0.011 0.011; visual sphere radius=0.001
- added link feet_fr, mass 0.010; collision box size=0.011 0.011 0.011; visual sphere radius=0.001
- added link femur_bl_link, mass 0.084; collision mesh filename=/home/ajoymathew07/Catatron/Catatron/src/catatron_descripti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; visual mesh filename=/home/ajoymathew07/Catatron/Catatron/src/catatron_descripti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
- added link femur_br_link, mass 0.084; collision mesh filename=/home/ajoymathew07/Catatron/Catatron/src/catatron_descripti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; visual mesh filename=/home/ajoymathew07/Catatron/Catatron/src/catatron_descripti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
- added link femur_fl_link, mass 0.084; collision mesh filename=/home/ajoymathew07/Catatron/Catatron/src/catatron_descripti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; visual mesh filename=/home/ajoymathew07/Catatron/Catatron/src/catatron_descripti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
- added link femur_fr_link, mass 0.084; collision mesh filename=/home/ajoymathew07/Catatron/Catatron/src/catatron_descripti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; visual mesh filename=/home/ajoymathew07/Catatron/Catatron/src/catatron_descripti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
- added link hip_bl_link, mass 0.233; collision mesh filename=/home/ajoymathew07/Catatron/Catatron/src/catatron_descripti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; visual mesh filename=/home/ajoymathew07/Catatron/Catatron/src/catatron_descripti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
- added link hip_bl_ref, mass 0.001; collision box size=0.002 0.002 0.002; visual box size=0.002 0.002 0.002
- added link hip_br_link, mass 0.233; collision mesh filename=/home/ajoymathew07/Catatron/Catatron/src/catatron_descripti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; visual mesh filename=/home/ajoymathew07/Catatron/Catatron/src/catatron_descripti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
- added link hip_br_ref, mass 0.001; collision box size=0.002 0.002 0.002; visual box size=0.002 0.002 0.002
- added link hip_fl_link, mass 0.233; collision mesh filename=/home/ajoymathew07/Catatron/Catatron/src/catatron_descripti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; visual mesh filename=/home/ajoymathew07/Catatron/Catatron/src/catatron_descripti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
- added link hip_fl_ref, mass 0.001; collision box size=0.002 0.002 0.002; visual box size=0.002 0.002 0.002
- added link hip_fr_link, mass 0.233; collision mesh filename=/home/ajoymathew07/Catatron/Catatron/src/catatron_descripti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; visual mesh filename=/home/ajoymathew07/Catatron/Catatron/src/catatron_descripti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
- added link hip_fr_ref, mass 0.001; collision box size=0.002 0.002 0.002; visual box size=0.002 0.002 0.002
- added link imu_link, mass 0.05; collision box size=0.05 0.05 0.01; visual box size=0.05 0.05 0.01
- added link tibia_bl_link, mass 0.034; collision mesh filename=/home/ajoymathew07/Catatron/Catatron/src/catatron_descripti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; visual mesh filename=/home/ajoymathew07/Catatron/Catatron/src/catatron_descripti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
- added link tibia_br_link, mass 0.034; collision mesh filename=/home/ajoymathew07/Catatron/Catatron/src/catatron_descripti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; visual mesh filename=/home/ajoymathew07/Catatron/Catatron/src/catatron_descripti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
- added link tibia_fl_link, mass 0.034; collision mesh filename=/home/ajoymathew07/Catatron/Catatron/src/catatron_descripti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; visual mesh filename=/home/ajoymathew07/Catatron/Catatron/src/catatron_descripti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
- added link tibia_fr_link, mass 0.034; collision mesh filename=/home/ajoymathew07/Catatron/Catatron/src/catatron_descripti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; visual mesh filename=/home/ajoymathew07/Catatron/Catatron/src/catatron_descripti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
- link base_link: mass 0.81776 -> 2.000; geometry collision mesh filename=/home/ajoymathew07/Catatron/Catatron/src/catatron_descripti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; visual mesh filename=/home/ajoymathew07/Catatron/Catatron/src/catatron_descripti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
Joints:
- removed joint FL1_joint
- removed joint FL2_joint
- removed joint FL3_joint
- removed joint FL4_joint
- removed joint FR1_joint
- removed joint FR2_joint
- removed joint FR3_joint
- removed joint FR4_joint
- removed joint RL1_joint
- removed joint RL2_joint
- removed joint RL3_joint
- removed joint RL4_joint
- removed joint RR1_joint
- removed joint RR2_joint
- removed joint RR3_joint
- removed joint RR4_joint
- removed joint world_to_base
- added joint bl_ref: type fixed, parent base_link, child hip_bl_ref, origin xyz=-0.09170 0.05355 -0.00279
- added joint br_ref: type fixed, parent base_link, child hip_br_ref, origin xyz=-0.09170 -0.05355 -0.00279
- added joint feet_bl_ref: type fixed, parent tibia_bl_link, child feet_bl, origin xyz=0.00000 -0.00834 -0.10000
- added joint feet_br_ref: type fixed, parent tibia_br_link, child feet_br, origin xyz=0.00000 0.00834 -0.10000
- added joint feet_fl_ref: type fixed, parent tibia_fl_link, child feet_fl, origin xyz=0.00000 -0.00834 -0.10000
- added joint feet_fr_ref: type fixed, parent tibia_fr_link, child feet_fr, origin xyz=0.00000 0.00834 -0.10000
- added joint fl_ref: type fixed, parent base_link, child hip_fl_ref, origin xyz=0.09170 0.05355 -0.00279
- added joint fr_ref: type fixed, parent base_link, child hip_fr_ref, origin xyz=0.09170 -0.05355 -0.00279
- added joint hip1_bl: type revolute, parent hip_bl_ref, child hip_bl_link, origin xyz=0.00000 0.00000 0.00000, axis 1.000 0.000 0.000, limit lower=-3.142 upper=3.142 effort=80.00000 velocity=1.04720
- added joint hip1_br: type revolute, parent hip_br_ref, child hip_br_link, origin xyz=0.00000 0.00000 0.00000, axis 1.000 0.000 0.000, limit lower=-3.142 upper=3.142 effort=80.00000 velocity=1.04720
- added joint hip1_fl: type revolute, parent hip_fl_ref, child hip_fl_link, origin xyz=0.00000 0.00000 0.00000, axis 1.000 0.000 0.000, limit lower=-3.142 upper=3.142 effort=80.00000 velocity=1.04720
- added joint hip1_fr: type revolute, parent hip_fr_ref, child hip_fr_link, origin xyz=0.00000 0.00000 0.00000, axis 1.000 0.000 0.000, limit lower=-3.142 upper=3.142 effort=80.00000 velocity=1.04720
- added joint hip2_bl: type revolute, parent hip_bl_link, child femur_bl_link, origin xyz=0.00000 0.03559 0.00000, axis 0.000 1.000 0.000, limit lower=-3.142 upper=3.142 effort=80.00000 velocity=1.04720
- added joint hip2_br: type revolute, parent hip_br_link, child femur_br_link, origin xyz=0.00000 -0.03559 0.00000, axis 0.000 1.000 0.000, limit lower=-3.142 upper=3.142 effort=80.00000 velocity=1.04720
- added joint hip2_fl: type revolute, parent hip_fl_link, child femur_fl_link, origin xyz=0.00000 0.03559 0.00000, axis 0.000 1.000 0.000, limit lower=-3.142 upper=3.142 effort=80.00000 velocity=1.04720
- added joint hip2_fr: type revolute, parent hip_fr_link, child femur_fr_link, origin xyz=0.00000 -0.03559 0.00000, axis 0.000 1.000 0.000, limit lower=-3.142 upper=3.142 effort=80.00000 velocity=1.04720
- added joint imu_joint: type fixed, parent base_link, child imu_link, origin xyz=0.0 0.0 0.06 rpy=0 0 0
- added joint knee_bl: type revolute, parent femur_bl_link, child tibia_bl_link, origin xyz=0.00000 0.01071 -0.09996, axis 0.000 1.000 0.000, limit lower=-3.142 upper=-0.52360 effort=80.00000 velocity=1.04720
- added joint knee_br: type revolute, parent femur_br_link, child tibia_br_link, origin xyz=0.00000 -0.01071 -0.09996, axis 0.000 1.000 0.000, limit lower=-3.142 upper=-0.52360 effort=80.00000 velocity=1.04720
- added joint knee_fl: type revolute, parent femur_fl_link, child tibia_fl_link, origin xyz=0.00000 0.01071 -0.09996, axis 0.000 1.000 0.000, limit lower=-3.142 upper=-0.52360 effort=80.00000 velocity=1.04720
- added joint knee_fr: type revolute, parent femur_fr_link, child tibia_fr_link, origin xyz=0.00000 -0.01071 -0.09996, axis 0.000 1.000 0.000, limit lower=-3.142 upper=-0.52360 effort=80.00000 velocity=1.04720
